File: oakram.sch (KiCad schematic (older format))
At the start: 11 parts, among them U1 IS41C16105C, U2 IS41C16105C, X1 ZIP40, X2 ZIP40

Commit message: Messing around with grounding etc
Parts:
- C1, C2, C3, C4, C5, C6: symbol C -> Device:C
- C7: symbol CP1 -> Device:CP1
- U1, U2: symbol DRAM_1MX16_SOJ -> oakram-rescue:DRAM_1MX16_SOJ
- X1, X2: symbol ZIP40 -> oakram:ZIP40
Connections:
- net labels added: ~OE1, ~OE2
- net labels removed: ~OE
- wire segments 84 -> 96
Changed lines of the file:
@@
-EESchema Schematic File Version 2
-LIBS:power
-LIBS:device
-LIBS:transistors
-LIBS:conn
-LIBS:linear
-LIBS:regul
-LIBS:74xx
-LIBS:cmos4000
-LIBS:adc-dac
-LIBS:memory
-LIBS:xilinx
-LIBS:microcontrollers
-LIBS:dsp
-LIBS:microchip
-LIBS:analog_switches
-LIBS:motorola
-LIBS:texas
-LIBS:intel
-LIBS:audio
-LIBS:interface
-LIBS:digital-audio
-LIBS:philips
-LIBS:display
-LIBS:cypress
-LIBS:siliconi
-LIBS:opto
-LIBS:atmel
-LIBS:contrib
-LIBS:valves
-LIBS:oakram
+EESchema Schematic File Version 4
 LIBS:oakram-cache
 EELAYER 26 0
@@
 $EndDescr
 $Comp
-L ZIP40 X1
+L oakram:ZIP40 X1
 U 1 1 59C97991
 P 4350 1800
@@
 	3950 2650 3600 2650
 Text Label 3600 2650 2    60   ~ 0
-~OE
+~OE1
 Wire Wire Line
 	3950 2750 3600 2750
@@
 ~CAS1
 $Comp
-L ZIP40 X2
+L oakram:ZIP40 X2
 U 1 1 59C9833A
 P 4350 4125
@@
 	3950 4975 3600 4975
 Text Label 3600 4975 2    60   ~ 0
-~OE
+~OE2
 Wire Wire Line
 	3950 5075 3600 5075
@@
 $EndBitmap
 $Comp
-L DRAM_1MX16_SOJ U2
+L oakram-rescue:DRAM_1MX16_SOJ U2
 U 1 1 59C98680
 P 8550 1725
@@
 $EndComp
 $Comp
-L DRAM_1MX16_SOJ U1
+L oakram-rescue:DRAM_1MX16_SOJ U1
 U 1 1 59C98929
 P 8450 4375
@@
 ~WE
 Text Label 7650 5225 2    60   ~ 0
-~OE
+~OE2
 Text Label 7750 2575 2    60   ~ 0
-~OE
+~OE1
 Text Label 7750 2175 2    60   ~ 0
 ~RAS
@@
 VCC
 Wire Wire Line
-	2525 5975 6325 5975
+	2525 5975 2850 5975
 $Comp
-L C C1
+L Device:C C1
 U 1 1 59CBE190
 P 2850 6250
@@
 Connection ~ 2850 5975
 Wire Wire Line
-	2525 6575 6325 6575
+	2525 6575 2850 6575
 Wire Wire Line
 	2850 6400 2850 6575
 Connection ~ 2850 6575
 $Comp
-L C C2
+L Device:C C2
 U 1 1 59CBE35E
 P 3350 6250
@@
 $EndComp
 $Comp
-L C C3
+L Device:C C3
 U 1 1 59CBE39E
 P 3800 6250
@@
 $EndComp
 $Comp
-L C C4
+L Device:C C4
 U 1 1 59CBE4F8
 P 4325 6250
@@
 	4325 6400 4325 6575
 $Comp
-L C C5
+L Device:C C5
 U 1 1 59CBE500
 P 4825 6250
@@
 $EndComp
 $Comp
-L C C6
+L Device:C C6
 U 1 1 59CBE506
 P 5275 6250
@@
 Connection ~ 4325 5975
 $Comp
-L CP1 C7
+L Device:CP1 C7
 U 1 1 59CA5A3F
 P 6325 6300
@@
 	6325 5975 6325 6150
 Connection ~ 5275 5975
+Wire Wire Line
+	2850 5975 3350 5975
+Wire Wire Line
+	2850 6575 3350 6575
+Wire Wire Line
+	3350 5975 3800 5975
+Wire Wire Line
+	3350 6575 3800 6575
+Wire Wire Line
+	3800 5975 4325 5975
+Wire Wire Line
+	4825 5975 5275 5975
+Wire Wire Line
+	4825 6575 5275 6575
+Wire Wire Line
+	3800 6575 4325 6575
+Wire Wire Line
+	4325 6575 4825 6575
+Wire Wire Line
+	4325 5975 4825 5975
+Wire Wire Line
+	5275 6575 6325 6575
+Wire Wire Line
+	5275 5975 6325 5975
 $EndSCHEMATC
